File: pcb/rp2040-devboard.kicad_sch (KiCad schematic)
At the start: 0 parts

Commit message: finish routing
Changed lines of the file:
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@@
+	(wire
+		(pts
+			(xy 101.6 63.5) (xy 119.38 63.5)
+		)
+		(stroke
+			(width 0)
+			(type default)
+		)
+	)
 	(wire
 		(pts
@@
 	(wire
 		(pts
-			(xy 101.6 63.5) (xy 119.38 63.5)
-		)
-		(stroke
-			(width 0)
-			(type default)
-		)
-	)
-	(wire
-		(pts
 			(xy 168.91 88.9) (xy 187.96 88.9)
 		)
@@
 	(wire
 		(pts
+			(xy 168.91 66.04) (xy 187.96 66.04)
+		)
+		(stroke
+			(width 0)
+			(type default)
+		)
+	)
+	(wire
+		(pts
 			(xy 101.6 60.96) (xy 119.38 60.96)
-		)
-		(stroke
-			(width 0)
-			(type default)
-		)
-	)
-	(wire
-		(pts
-			(xy 168.91 66.04) (xy 187.96 66.04)
 		)
 		(stroke
@@
 		)
 		(pin "USB_D-" input
+			(at 119.38 63.5 180)
+			(effects
+				(font
+					(size 1.27 1.27)
+				)
+				(justify left)
+			)
+		)
+		(pin "USB_D+" input
 			(at 119.38 60.96 180)
 			(effects
 				(font
-					(size 1.27 1.27)
-				)
-				(justify left)
-			)
-		)
-		(pin "USB_D+" input
-			(at 119.38 63.5 180)
-			(effects
-				(font
